File: usb-booster.kicad_pcb (KiCad board)
At the start: 2 copper layers, 40 x 25 mm, 24 parts, among them J1 USB_C_Receptacle_USB2.0_16P, J2 Conn_01x02, U1 MC34063AD

Commit message: fix: GND label
Other:
- board text added: "GND"
- board text removed: "-12V"
